Commit message: feat: more more more

File: src/real_bot/description/lidar.xacro (robot description, xacro)
@@ -13,5 +13,5 @@
       <parent link="chassis"/>
       <child link="laser_frame"/>
-      <origin xyz="0.11 0 0.27" rpy="0 0 0"/>
+      <origin xyz="0.11 0 0.27" rpy="0 0 3.14159"/>
     </joint>
     <link name="laser_frame">
